File: hardware/kicad/WifiKiwi.kicad_pcb (KiCad board)
At the start: 4 copper layers, 0 parts

Commit message: Scaffold KiCad 10 hierarchical project
Builds out the KiCad project to a state that opens cleanly, exports to
PDF/SVG, passes DRC, and gives a human a structured starting point for
schematic capture and PCB layout.

hardware/kicad/
  - WifiKiwi.kicad_pro: KiCad 10 project with Default/RF50/Power
    net classes pre-configured.
  - WifiKiwi.kicad_sch: hierarchical root with 7 sheet symbols
    (Power, MCU, Display, RF front-end, Sub-GHz, Sig-Gen, I/O).
  - sheets/01..07_*.kicad_sch: per-subsystem sub-sheets, each with
    hierarchical pins matching the root and a netlist-plan text
    block describing what needs to be wired (rails, decoupling,
    pin assignments, RF topology, layout constraints).
  - WifiKiwi.kicad_pcb: 100x65 mm rectangular outline with 4
    mounting-hole pilots in the corners. Empty (no copper, no
    footprints) - layout is a follow-up task.
  - symbols/wifikiwi.kicad_sym: empty project-local symbol library
    stub (KiCad 10 format). README lists the 8 symbols a human
    still needs to draw with datasheet pinouts.
  - footprints/wifikiwi.pretty/: empty project-local footprint dir.
  - sym-lib-table, fp-lib-table: auto-mount the project libraries.
  - gen_sheets.py: regenerates sheets/* + root from a Python schema.
    Use only while iterating on sheet structure; clobbers GUI edits.
  - README.md: full documentation of layout, regen workflow, symbols
    TODO, gerber export commands, and net-class details.

Validation:
  - kicad-cli sch erc:    151 violations, all 'pin not connected'
                          on hierarchical sheet pins (expected; nets
                          unwired by design).
  - kicad-cli pcb drc:    0 violations, 0 unconnected items.
  - kicad-cli sch export pdf: succeeds (162 KB output).

.gitignore:
  - exclude KiCad runtime cruft (*.lck, *.kicad_prl, .history/,
    *-backups/, fp-info-cache).

Co-authored-by: Copilot <223556219+Copilot@users.noreply.github.com>
Signed-off-by: Ari Cummings <ari@aricummings.com>
Other:
- board outline added: 100 x 65 mm
- board text added: "Layout pending - see docs/plan.md"
- board text added: "WifiKiwi v0.1.0-dev"
Changed lines of the file:
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@@
-(kicad_pcb (version 20240108) (generator "wifikiwi-scaffold")
-  (general
-    (thickness 1.6)
-  )
-  (paper "A4")
-  (title_block
-    (title "WifiKiwi - PCB")
-    (rev "0.1.0-dev")
-    (company "WifiKiwi contributors")
-    (comment 1 "Layout pending - 4 layer stackup")
-    (comment 2 "Licensed under CERN-OHL-S v2")
-  )
-  (layers
-    (0 "F.Cu" signal)
-    (1 "In1.Cu" signal "GND")
-    (2 "In2.Cu" signal "PWR")
-    (31 "B.Cu" signal)
-    (32 "B.Adhes" user "B.Adhesive")
-    (33 "F.Adhes" user "F.Adhesive")
-    (34 "B.Paste" user)
-    (35 "F.Paste" user)
-    (36 "B.SilkS" user "B.Silkscreen")
-    (37 "F.SilkS" user "F.Silkscreen")
-    (38 "B.Mask" user)
-    (39 "F.Mask" user)
-    (40 "Dwgs.User" user "User.Drawings")
-    (41 "Cmts.User" user "User.Comments")
-    (44 "Edge.Cuts" user)
-    (45 "Margin" user)
-    (46 "B.CrtYd" user "B.Courtyard")
-    (47 "F.CrtYd" user "F.Courtyard")
-    (48 "B.Fab" user)
-    (49 "F.Fab" user)
-  )
-  (setup
-    (pad_to_mask_clearance 0)
-  )
-  (net 0 "")
+(kicad_pcb
+	(version 20260206)
+	(generator "pcbnew")
+	(generator_version "10.0")
+	(general
+		(thickness 1.6)
+		(legacy_teardrops no)
+	)
+	(paper "A4")
+	(title_block
+		(title "WifiKiwi - PCB")
+		(rev "0.1.0-dev")
+		(company "WifiKiwi contributors")
+		(comment 1 "100mm x 65mm 4-layer board, 1.6mm FR4")
+		(comment 2 "Layer stackup: TOP / GND / PWR / BOT")
+		(comment 3 "Licensed under CERN-OHL-S v2")
+	)
+	(layers
+		(0 "F.Cu" signal)
+		(4 "In1.Cu" signal "GND")
+		(6 "In2.Cu" signal "PWR")
+		(2 "B.Cu" signal)
+		(9 "F.Adhes" user "F.Adhesive")
+		(11 "B.Adhes" user "B.Adhesive")
+		(13 "F.Paste" user)
+		(15 "B.Paste" user)
+		(5 "F.SilkS" user "F.Silkscreen")
+		(7 "B.SilkS" user "B.Silkscreen")
+		(1 "F.Mask" user)
+		(3 "B.Mask" user)
+		(17 "Dwgs.User" user "User.Drawings")
+		(19 "Cmts.User" user "User.Comments")
+		(25 "Edge.Cuts" user)
+		(27 "Margin" user)
+		(31 "F.CrtYd" user "F.Courtyard")
+		(29 "B.CrtYd" user "B.Courtyard")
+		(35 "F.Fab" user)
+		(33 "B.Fab" user)
+	)
+	(setup
+		(pad_to_mask_clearance 0)
+		(allow_soldermask_bridges_in_footprints no)
+		(tenting
+			(front yes)
+			(back yes)
+		)
+		(covering
+			(front no)
+			(back no)
+		)
+		(plugging
+			(front no)
+			(back no)
+		)
+		(capping no)
+		(filling no)
+		(pcbplotparams
+			(layerselection 0x00000000_00000000_55555555_5755f5ff)
+			(plot_on_all_layers_selection 0x00000000_00000000_00000000_00000000)
+			(disableapertmacros no)
+			(usegerberextensions no)
+			(usegerberattributes yes)
+			(usegerberadvancedattributes yes)
+			(creategerberjobfile yes)
+			(dashed_line_dash_ratio 12)
+			(dashed_line_gap_ratio 3)
+			(svgprecision 4)
+			(plotframeref no)
+			(mode 1)
+			(useauxorigin no)
+			(pdf_front_fp_property_popups yes)
+			(pdf_back_fp_property_popups yes)
+			(pdf_metadata yes)
+			(pdf_single_document no)
+			(dxfpolygonmode yes)
+			(dxfimperialunits yes)
+			(dxfusepcbnewfont yes)
+			(psnegative no)
+			(psa4output no)
+			(plot_black_and_white yes)
+			(sketchpadsonfab no)
+			(plotpadnumbers no)
+			(hidednponfab no)
+			(sketchdnponfab yes)
+			(crossoutdnponfab yes)
+			(subtractmaskfromsilk no)
+			(outputformat 1)
+			(mirror no)
+			(drillshape 1)
+			(scaleselection 1)
+			(outputdirectory "")
+		)
+	)
+	(gr_line
+		(start 0 0)
+		(end 100 0)
+		(stroke
+			(width 0.1)
+			(type solid)
+		)
+		(layer "Edge.Cuts")
+	)
+	(gr_line
+		(start 0 65)
+		(end 0 0)
+		(stroke
+			(width 0.1)
+			(type solid)
+		)
+		(layer "Edge.Cuts")
+	)
+	(gr_circle
+		(center 4 4)
+		(end 5.6 4)
+		(stroke
+			(width 0.1)
+			(type solid)
+		)
+		(fill no)
+		(layer "Edge.Cuts")
+	)
+	(gr_circle
+		(center 4 61)
+		(end 5.6 61)
+		(stroke
+			(width 0.1)
+			(type solid)
+		)
+		(fill no)
+		(layer "Edge.Cuts")
+	)
+	(gr_circle
+		(center 96 4)
+		(end 97.6 4)
+		(stroke
+			(width 0.1)
+			(type solid)
+		)
+		(fill no)
+		(layer "Edge.Cuts")
+	)
+	(gr_circle
+		(center 96 61)
+		(end 97.6 61)
+		(stroke
+			(width 0.1)
+			(type solid)
+		)
+		(fill no)
+		(layer "Edge.Cuts")
+	)
+	(gr_line
+		(start 100 0)
+		(end 100 65)
+		(stroke
+			(width 0.1)
+			(type solid)
+		)
+		(layer "Edge.Cuts")
+	)
+	(gr_line
+		(start 100 65)
+		(end 0 65)
+		(stroke
+			(width 0.1)
+			(type solid)
+		)
+		(layer "Edge.Cuts")
+	)
+	(gr_text "Layout pending - see docs/plan.md"
+		(at 50 37 0)
+		(layer "F.SilkS")
+		(effects
+			(font
+				(size 1 1)
+				(thickness 0.15)
+			)
+		)
+	)
+	(gr_text "WifiKiwi v0.1.0-dev"
+		(at 50 32 0)
+		(layer "F.SilkS")
+		(effects
+			(font
+				(size 2 2)
+				(thickness 0.3)
+			)
+		)
+	)
+	(embedded_fonts no)
 )
