File: hardware/kicad/WifiKiwi.kicad_sch (KiCad schematic)
At the start: 0 parts

Commit message: Scaffold KiCad 10 hierarchical project
Builds out the KiCad project to a state that opens cleanly, exports to
PDF/SVG, passes DRC, and gives a human a structured starting point for
schematic capture and PCB layout.

hardware/kicad/
  - WifiKiwi.kicad_pro: KiCad 10 project with Default/RF50/Power
    net classes pre-configured.
  - WifiKiwi.kicad_sch: hierarchical root with 7 sheet symbols
    (Power, MCU, Display, RF front-end, Sub-GHz, Sig-Gen, I/O).
  - sheets/01..07_*.kicad_sch: per-subsystem sub-sheets, each with
    hierarchical pins matching the root and a netlist-plan text
    block describing what needs to be wired (rails, decoupling,
    pin assignments, RF topology, layout constraints).
  - WifiKiwi.kicad_pcb: 100x65 mm rectangular outline with 4
    mounting-hole pilots in the corners. Empty (no copper, no
    footprints) - layout is a follow-up task.
  - symbols/wifikiwi.kicad_sym: empty project-local symbol library
    stub (KiCad 10 format). README lists the 8 symbols a human
    still needs to draw with datasheet pinouts.
  - footprints/wifikiwi.pretty/: empty project-local footprint dir.
  - sym-lib-table, fp-lib-table: auto-mount the project libraries.
  - gen_sheets.py: regenerates sheets/* + root from a Python schema.
    Use only while iterating on sheet structure; clobbers GUI edits.
  - README.md: full documentation of layout, regen workflow, symbols
    TODO, gerber export commands, and net-class details.

Validation:
  - kicad-cli sch erc:    151 violations, all 'pin not connected'
                          on hierarchical sheet pins (expected; nets
                          unwired by design).
  - kicad-cli pcb drc:    0 violations, 0 unconnected items.
  - kicad-cli sch export pdf: succeeds (162 KB output).

.gitignore:
  - exclude KiCad runtime cruft (*.lck, *.kicad_prl, .history/,
    *-backups/, fp-info-cache).

Co-authored-by: Copilot <223556219+Copilot@users.noreply.github.com>
Signed-off-by: Ari Cummings <ari@aricummings.com>
Other:
- added sheet Display - ILI9488 3.5" SPI LCD + FT6336U cap touch (sheets/03_display.kicad_sch)
- added sheet MCU - ESP32-C5-WROOM-1U + USB/JTAG + boot logic (sheets/02_mcu.kicad_sch)
- added sheet Power - USB-C input, charger, regulators (sheets/01_power.kicad_sch)
- added sheet RF Front-End - SMA-A/B, diplexer, 3x PE4259, 2x PE43711, 2x SPF5189Z, U.FL test pads, bias-T (sheets/04_rf_frontend.kicad_sch)
- added sheet Signal generator - ADF4351 PLL/VCO (sheets/06_siggen.kicad_sch)
- added sheet Sub-GHz - CC1101 transceiver (sheets/05_subghz.kicad_sch)
- added sheet User I/O - buttons, RGB LED, RF-active LED, MicroSD (sheets/07_io.kicad_sch)
